File: machxo5.kicad_sch (KiCad schematic)
At the start: 129 parts, among them J3001 PinHeader_2x5_P1.27mm_SMD, J3002 PinHeader_2x5_P1.27mm_SMD, J3003 PinHeader_2x5_P1.27mm_SMD, J3004 PinHeader_2x5_P1.27mm_SMD, J3005 PinHeader_2x5_P1.27mm_SMD, J3006 PinHeader_2x5_P1.27mm_SMD, J3007 PinHeader_2x5_P1.27mm_SMD, J3008 PinHeader_2x5_P1.27mm_SMD, J3009 PinHeader_2x5_P1.27mm_SMD, J3010 PinHeader_2x5_P1.27mm_SMD, J3011 PinHeader_2x5_P1.27mm_SMD, SW3001 SW_KSC441J70SHLFS_SMD, SW3002 SW_KSC441J70SHLFS_SMD, SW3004 SW_KSC441J70SHLFS_SMD, U3001 LFMXO5-25-7BBG400C, Y3001 Resonator_32.768kHz_ECX-31B, Y3002 Oscillator_125MHz_ASEMB

Commit message: [#103910] Complete schematics
Parts:
- removed C3001, C3014, C3015: C_1u_0603, antmicro-footprints:C_0603_1608Metric, symbol antmicroCapacitors0603:C_1u_0603
- removed C3002, C3003: C_22p_0402, antmicro-footprints:C_0402_1005Metric, symbol antmicroCapacitors0402:C_22p_0402
- removed C3004, C3005, C3006, C3007, C3011, C3012: C_100n_0402, antmicro-footprints:C_0402_1005Metric, symbol antmicroCapacitors0402:C_100n_0402
- removed C3008, C3009: C_100n_16V_X7R_0402, antmicro-footprints:C_0402_1005Metric, symbol antmicroCapacitors0402:C_100n_16V_X7R_0402
- removed C3013: C_1u_6.3V_X6S_0402, antmicro-footprints:C_0402_1005Metric, symbol antmicroCapacitors0402:C_1u_6.3V_X6S_0402
- removed D3001, D3002: BAT54-02V-G3-08, antmicro-footprints:SOD-523, symbol antmicroDiodesRectifiersSingle:BAT54-02V-G3-08
- removed R3003, R3037: R_1k_0402, antmicro-footprints:R_0402_1005Metric, symbol antmicroResistors0402:R_1k_0402
- removed R3005, R3025, R3029, R3030, R3031, R3032, R3033, R3034, R3035, R3036, R3049: R_10k_0402, antmicro-footprints:R_0402_1005Metric, symbol antmicroResistors0402:R_10k_0402
- removed R3006: R_100R_0402, antmicro-footprints:R_0402_1005Metric, symbol Antmicro Symbols:R_100R_0402
- removed R3007, R3008, R3009, R3010, R3011, R3012, R3013, R3014, R3015, R3016, R3017, R3018, R3019, R3020, R3021, R3022, R3023, R3024: R_4k7_0402, antmicro-footprints:R_0402_1005Metric, symbol antmicroResistors0402:R_4k7_0402
- removed R3038, R3039, R3040: R_100k_0402, antmicro-footprints:R_0402_1005Metric, symbol antmicroResistors0402:R_100k_0402
- removed R3041, R3042, R3043, R3044, R3045, R3046, R3047: R_0R_0402, antmicro-footprints:R_0402_1005Metric, symbol antmicroResistors0402:R_0R_0402
- removed SW3002: SW_KSC441J70SHLFS_SMD, antmicro-footprints:SW_KSC441J70SHLFS_SMD, symbol antmicroPushbuttonSwitches:SW_KSC441J70SHLFS_SMD
- removed TP3002, TP3003, TP3004, TP3005, TP3006, TP3007, TP3010: TP_1mm_SMD, antmicro-footprints:TP_SMD_1mm, symbol antmicroTestPoints:TP_1mm_SMD
- removed Y3001: Resonator_32.768kHz_ECX-31B, antmicro-footprints:Resonator_SMD_ECS_ECX-31B_3.2x1.5x0.9mm, symbol antmicroResonators:Resonator_32.768kHz_ECX-31B
- added C? (x10): C_100n_0402, antmicro-footprints:C_0402_1005Metric, symbol antmicroCapacitors0402:C_100n_0402
- added J? (x2): PinHeader_2x5_P1.27mm_SMD, antmicro-footprints:PinHeader_2x5_P1.27mm_SMD, symbol antmicroGenericPinHeaders:PinHeader_2x5_P1.27mm_SMD
Connections:
- net nRESET_IN is gone; now on net ~{BTN0}: C3010.2, R3001.2, R3002.1
- net +1V8: now also U3001.[T12,V14] (VCCIO5), U3001.[T9,V8] (VCCIO6), C?.2, C?.2, C?.2, C?.2, J?.6
- net +3V3: now also U3001.[F2,H4] (VCCIO9), U3001.[L18,M15] (VCCIO3), U3001.[R18,U17] (VCCIO4), C?.2, C?.2, C?.2, C?.2, C?.2, C?.2, J?.6
- net 7SEG_L.A: now also U3001.H19 (PR13A)
- net 7SEG_L.B: now also U3001.H20 (PR13B)
- net 7SEG_L.C: now also U3001.H13 (PR14A)
- net 7SEG_L.D: now also U3001.J12 (PR14B)
- net 7SEG_L.DP: now also U3001.J16 (PR16B)
- net 7SEG_L.E: now also U3001.J13 (PR15A)
- net 7SEG_L.F: now also U3001.J14 (PR15B)
- net 7SEG_L.G: now also U3001.J15 (PR16A)
- net GND: now also SW3001.3, SW3004.3, U3001.W15 (ADC_REFP0), U3001.Y15 (ADC_REFP1), U3001.Y16 (ADC_DP0), U3001.Y17 (ADC_DN0), U3001.Y18 (ADC_DP1), U3001.Y19 (ADC_DN1), C?.1, C?.1, C?.1, C?.1, C?.1, C?.1, C?.1, C?.1, C?.1, C?.1, J?.5, J?.5
- net PWRGD_S0iX: no longer R3028.1
- net ~{PROGRAM}: now also R3028.1
- net PL2A: now reaches U3001.B1 (PL2A/ULC_GPLL0T_IN)
- net PL2A: now also J?.1
- net PL2B: now reaches U3001.C1 (PL2B)
- net PL2B: now also J?.3
- net PL3B: now reaches U3001.D1 (PL3B)
- net PL3B: now also J?.9
- net PL3A: now reaches U3001.D2 (PL3A)
- net PL3A: now also J?.7
- net PL5A: now reaches U3001.E1 (PL5A)
- net PL5A: now also J?.8
- net PL4B: now reaches U3001.E2 (PL4B)
- net PL4B: now also J?.4
- net PL4A: now reaches U3001.E3 (PL4A)
- net PL4A: now also J?.2
- net PL5B: now reaches U3001.F1 (PL5B)
- net PL5B: now also J?.10
- net ~{BTN0}: now reaches U3001.P3 (PL34A)
- net at SW3001.1: now also R3002.2, SW3001.2
- net at SW3004.1: now also R3027.2, SW3004.2
- net PT9A: now reaches U3001.A2 (PT9A)
- net PT9A: now also J?.7
- net PT9B: now reaches U3001.A3 (PT9B)
- net PT9B: now also J?.9
- net PT11B: now reaches U3001.A4 (PT11B)
- net PT11B: now also J?.10
- net PT8B: now reaches U3001.B2 (PT8B)
- net PT8B: now also J?.3
- net PT11A: now reaches U3001.B3 (PT11A)
- net PT11A: now also J?.8
- net PT8A: now reaches U3001.C2 (PT8A)
- net PT8A: now also J?.1
- net PT10B: now reaches U3001.C3 (PT10B)
- net PT10B: now also J?.4
- net PT10A: now reaches U3001.D3 (PT10A)
- net PT10A: now also J?.2
- no-connect marks 269 -> 244
Other:
- note removed: "Boot Source Select Strap: - 1(R3003 not mounted)=Use the shared SPI pins for boot - 0(R3003 mounted)=Use the eSPI Flash Channel for boot"
- note removed: "C3001 max. ESR = 100mohm"
- note removed: "I2C channels: 01-07"
- note removed: "JTAG_STRAP"
- note removed: "PVT Flash"
- note removed: "SPI Flash used - ~{RSMRST} signal can be on any GPIO"
- moved on the sheet: C3010, C3018, C3023, C3024, C3025, C3026, C3027, C3028, C3029, R3001, R3002, R3004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

Commit message: [#103910] Annotate schematics & Clean ERC
Parts:
- removed J3001, J3002, J3003, J3004, J3005, J3006, J3007, J3008, J3009, J3010, J3011: PinHeader_2x5_P1.27mm_SMD, antmicro-footprints:PinHeader_2x5_P1.27mm_SMD, symbol antmicroGenericPinHeaders:PinHeader_2x5_P1.27mm_SMD
- R3002, R3027: symbol Antmicro Symbols:R_100R_0402 -> antmicroResistors0402:R_100R_0402
- gave numbers to parts that had none: 12
Connections:
- net FPGA_JTAG.TRST: now also U3001.G17 (PR8B/SD11)
- no-connect marks 244 -> 239
Other:
- note removed: "PIN BREAKOUT"

Commit message: [#103953] sch/pcb: re-annotate components
Parts:
- renumbered C3020 to C1, C3032 to C10, C3035 to C11, C3039 to C12, C3043 to C13, C3046 to C14, C3049 to C15, C3033 to C16, C3036 to C17, C3040 to C18, C3044 to C19, C3021 to C2, C3047 to C20, C3034 to C21, C3037 to C22, C3041 to C23, C3016 to C24, C3017 to C25, C3019 to C26, C3023 to C27, C3001 to C28, C3026 to C29, C3022 to C3, C3002 to C30, C3018 to C31, C3010 to C32, C3003 to C33, C3004 to C34, C3005 to C35, C3006 to C36, C3024 to C37, C3007 to C38, C3025 to C39, C3030 to C4, C3008 to C40, C3028 to C41, C3009 to C42, C3029 to C43, C3011 to C44, C3027 to C45, C3031 to C5, C3038 to C6, C3042 to C7, C3045 to C8, C3048 to C9, FB3001 to FB1, FB3002 to FB2, FB3003 to FB3, FB3004 to FB4, J3012 to J2, J3013 to J3, R3050 to R10, R3004 to R11, R3028 to R12, R3026 to R13, R3027 to R14, R3001 to R15, R3002 to R16, R3048 to R9, SW3004 to SW1, SW3001 to SW2, U3001 to U1, Y3002 to Y1
