File: power.kicad_sch (KiCad schematic)
At the start: 31 parts, among them Q4001 DMG1012T-7, U4001 AP62301_TSOT, U4002 TLV76701_WSON

Commit message: [#103910] Update power section
Parts:
- removed R4001: R_10k_0402, antmicro-footprints:R_0402_1005Metric, symbol antmicroResistors0402:R_10k_0402
- added C?: C_22u_16V_0603, antmicro-footprints:C_0603_1608Metric_EIA, symbol antmicroCapacitors0603:C_22u_16V_0603
- added C?: C_22u_0603, antmicro-footprints:C_0603_1608Metric, symbol antmicroCapacitors0603:C_22u_0603
- added C?: C_100n_50V_X8L_0402, antmicro-footprints:C_0402_1005Metric, symbol antmicroCapacitors0402:C_100n_50V_X8L_0402
- added C?: C_10u_16V_0603, antmicro-footprints:C_0603_1608Metric, symbol antmicroCapacitors0603:C_10u_16V_0603
- added D?: LED_G_0603_LTST-C190GKT, antmicro-footprints:LED_0603_1608Metric_G, symbol antmicroLEDIndicationDiscrete:LED_G_0603_LTST-C190GKT
- added L?: L_1u5_4.4A_Bourns-SRP3212A, antmicro-footprints:L_Bourns-SRP3212A, symbol antmicroFixedInductors:L_1u5_4.4A_Bourns-SRP3212A
- added Q?: DMG1012T-7, antmicro-footprints:SOT-523, symbol antmicroTransistorsFETsMOSFETsSingle:DMG1012T-7
- added R? (x3): R_10k_0402, antmicro-footprints:R_0402_1005Metric, symbol antmicroResistors0402:R_10k_0402
- added R? (x3): R_1k_0402, antmicro-footprints:R_0402_1005Metric, symbol antmicroResistors0402:R_1k_0402
- added R?: R_0R_0402, antmicro-footprints:R_0402_1005Metric, symbol antmicroResistors0402:R_0R_0402
- added R?: R_0R_22.4A_0603, antmicro-footprints:R_0603_1608Metric, symbol antmicroResistors0603:R_0R_22.4A_0603
- added R?: R_1k5_0402, antmicro-footprints:R_0402_1005Metric, symbol antmicroResistors0402:R_1k5_0402
- added TP?: TP_0.75mm_SMD, antmicro-footprints:TP_SMD_0.75mm, symbol antmicroTestPoints:TP_0.75mm_SMD
- added U?: AP62301_TSOT, antmicro-footprints:TSOT23-6, symbol antmicroDCDCConverters:AP62301_TSOT
- R4002, R4004, R4006: now fitted
- R4003, R4005: now not fitted; now in the parts list
Connections:
- net +3V3: now also R?.2
- net DC_SCM_STBY_EN: now also R?.1
- net GND: now also C?.1, C?.1, C?.1, Q?.2 (S), R?.1, R?.1, U?.1 (GND)
- net at D4001.2 (A): now also R?.1
- net DC_SCM_12V_AUX renamed VIN
- net VIN: now also C?.2, R?.2, R?.2, U?.3 (VIN)
- new net: D?.1 (C), Q?.3 (D)
- new net: D?.2 (A), R?.1
- new net: R?.1, R?.2
- new net +1V0: Q?.1 (G), R?.2, TP?.1
- new net 1V0_OUT: C?.2, C?.2, L?.2, R?.1, R?.2
- new net BST_1V0: C?.1, U?.6 (BST)
- new net EN_1V0: R?.1, R?.2, R?.2, U?.5 (EN)
- new net FB_1V0: R?.1, R?.2, U?.4 (FB)
- new net SW_1V0: C?.2, L?.1, U?.2 (SW)
Other:
- note added: "+1V0 DC/DC (MachXO5 V_{core})"
- note added: "+3V3 DC/DC"
- note added: "1V0 @ 3A"
- note removed: "+3V3 DC/DC converter"
- moved on the sheet: C4001, C4002, C4003, C4004, C4005, C4006, D4001, D4003, D4004, L4001, Q4001, R4007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

Commit message: [#103910] Annotate schematics & Clean ERC
Parts:
- gave numbers to parts that had none: 18
Changed lines of the file:
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@@
 		(in_pos_files yes)
 		(dnp no)
-		(property "Reference" "C?"
+		(property "Reference" "C4009"
 			(at 191.008 90.678 90)
 			(show_name no)
@@
 			(project "machxo5-espi-debugger"
 				(path "/df391740-647e-4ab6-9dcd-d61184d66fe9/1d07191d-71e0-43c8-9a4f-6404f7e36093"
-					(reference "C?")
+					(reference "C4009")
 					(unit 1)
 				)
@@
 		(in_pos_files yes)
 		(dnp no)
-		(property "Reference" "C?"
+		(property "Reference" "C4010"
 			(at 198.628 90.678 90)
 			(show_name no)
@@
 			(project "machxo5-espi-debugger"
 				(path "/df391740-647e-4ab6-9dcd-d61184d66fe9/1d07191d-71e0-43c8-9a4f-6404f7e36093"
-					(reference "C?")
+					(reference "C4010")
 					(unit 1)
 				)
@@
 		(dnp no)
 		(fields_autoplaced yes)
-		(property "Reference" "Q?"
+		(property "Reference" "Q4002"
 			(at 267.97 158.75 0)
 			(show_name no)
@@
 			(project "machxo5-espi-debugger"
 				(path "/df391740-647e-4ab6-9dcd-d61184d66fe9/1d07191d-71e0-43c8-9a4f-6404f7e36093"
-					(reference "Q?")
+					(reference "Q4002")
 					(unit 1)
 				)
@@
 		(dnp no)
 		(fields_autoplaced yes)
-		(property "Reference" "TP?"
+		(property "Reference" "TP4003"
 			(at 229.87 88.9 0)
 			(show_name no)
@@
 			(project "machxo5-espi-debugger"
 				(path "/df391740-647e-4ab6-9dcd-d61184d66fe9/1d07191d-71e0-43c8-9a4f-6404f7e36093"
-					(reference "TP?")
+					(reference "TP4003")
 					(unit 1)
 				)
@@
 		(in_pos_files yes)
 		(dnp no)
-		(property "Reference" "C?"
+		(property "Reference" "C4008"
 			(at 163.83 92.71 0)
 			(show_name no)
@@
 			(project "machxo5-espi-debugger"
 				(path "/df391740-647e-4ab6-9dcd-d61184d66fe9/1d07191d-71e0-43c8-9a4f-6404f7e36093"
-					(reference "C?")
+					(reference "C4008")
 					(unit 1)
 				)
@@
 		(in_pos_files yes)
 		(dnp no)
-		(property "Reference" "D?"
+		(property "Reference" "D4002"
 			(at 266.065 148.59 90)
 			(show_name no)
@@
 			(project "machxo5-espi-debugger"
 				(path "/df391740-647e-4ab6-9dcd-d61184d66fe9/1d07191d-71e0-43c8-9a4f-6404f7e36093"
-					(reference "D?")
+					(reference "D4002")
 					(unit 1)
 				)
@@
 		(dnp no)
 		(fields_autoplaced yes)
-		(property "Reference" "R?"
+		(property "Reference" "R4021"
 			(at 180.34 105.41 90)
 			(show_name no)
@@
 			(project "machxo5-espi-debugger"
 				(path "/df391740-647e-4ab6-9dcd-d61184d66fe9/1d07191d-71e0-43c8-9a4f-6404f7e36093"
-					(reference "R?")
+					(reference "R4021")
 					(unit 1)
 				)
@@
 		(dnp no)
 		(fields_autoplaced yes)
-		(property "Reference" "R?"
+		(property "Reference" "R4024"
 			(at 266.7 140.97 90)
 			(show_name no)
@@
 			(project "machxo5-espi-debugger"
 				(path "/df391740-647e-4ab6-9dcd-d61184d66fe9/1d07191d-71e0-43c8-9a4f-6404f7e36093"
-					(reference "R?")
+					(reference "R4024")
 					(unit 1)
 				)
@@
 		(dnp no)
 		(fields_autoplaced yes)
-		(property "Reference" "R?"
+		(property "Reference" "R4020"
 			(at 180.34 97.79 90)
 			(show_name no)
@@
 			(project "machxo5-espi-debugger"
 				(path "/df391740-647e-4ab6-9dcd-d61184d66fe9/1d07191d-71e0-43c8-9a4f-6404f7e36093"
-					(reference "R?")
+					(reference "R4020")
 					(unit 1)
 				)
@@
 		(dnp no)
 		(fields_autoplaced yes)
-		(property "Reference" "L?"
+		(property "Reference" "L4002"
 			(at 172.72 83.82 0)
 			(show_name no)
@@
 			(project "machxo5-espi-debugger"
 				(path "/df391740-647e-4ab6-9dcd-d61184d66fe9/1d07191d-71e0-43c8-9a4f-6404f7e36093"
-					(reference "L?")
+					(reference "L4002")
 					(unit 1)
 				)
@@
 		(dnp no)
 		(fields_autoplaced yes)
-		(property "Reference" "C?"
+		(property "Reference" "C4007"
 			(at 86.36 92.7036 90)
 			(show_name no)
@@
 			(project "machxo5-espi-debugger"
 				(path "/df391740-647e-4ab6-9dcd-d61184d66fe9/1d07191d-71e0-43c8-9a4f-6404f7e36093"
-					(reference "C?")
+					(reference "C4007")
 					(unit 1)
 				)
@@
 		(in_pos_files yes)
 		(dnp yes)
-		(property "Reference" "R?"
+		(property "Reference" "R4001"
 			(at 107.95 96.52 0)
 			(show_name no)
@@
 			(project "machxo5-espi-debugger"
 				(path "/df391740-647e-4ab6-9dcd-d61184d66fe9/1d07191d-71e0-43c8-9a4f-6404f7e36093"
-					(reference "R?")
+					(reference "R4001")
 					(unit 1)
 				)
@@
 		(dnp no)
 		(fields_autoplaced yes)
-		(property "Reference" "U?"
+		(property "Reference" "U4003"
 			(at 139.7 81.28 0)
 			(show_name no)
@@
 			(project "machxo5-espi-debugger"
 				(path "/df391740-647e-4ab6-9dcd-d61184d66fe9/1d07191d-71e0-43c8-9a4f-6404f7e36093"
-					(reference "U?")
+					(reference "U4003")
 					(unit 1)
 				)
@@
 		(dnp no)
 		(fields_autoplaced yes)
-		(property "Reference" "R?"
+		(property "Reference" "R4022"
 			(at 187.96 153.67 90)
 			(show_name no)
@@
 			(project "machxo5-espi-debugger"
 				(path "/df391740-647e-4ab6-9dcd-d61184d66fe9/1d07191d-71e0-43c8-9a4f-6404f7e36093"
-					(reference "R?")
+					(reference "R4022")
 					(unit 1)
 				)
@@
 		(in_pos_files yes)
 		(dnp yes)
-		(property "Reference" "R?"
+		(property "Reference" "R4010"
 			(at 121.92 100.33 90)
 			(show_name no)
@@
 			(project "machxo5-espi-debugger"
 				(path "/df391740-647e-4ab6-9dcd-d61184d66fe9/1d07191d-71e0-43c8-9a4f-6404f7e36093"
-					(reference "R?")
+					(reference "R4010")
 					(unit 1)
 				)
@@
 		(in_pos_files yes)
 		(dnp no)
-		(property "Reference" "R?"
+		(property "Reference" "R4023"
 			(at 208.28 86.36 0)
 			(show_name no)
@@
 			(project "machxo5-espi-debugger"
 				(path "/df391740-647e-4ab6-9dcd-d61184d66fe9/1d07191d-71e0-43c8-9a4f-6404f7e36093"
-					(reference "R?")
+					(reference "R4023")
 					(unit 1)
 				)
@@
 		(dnp no)
 		(fields_autoplaced yes)
-		(property "Reference" "R?"
+		(property "Reference" "R4019"
 			(at 180.34 91.44 90)
 			(show_name no)
@@
 			(project "machxo5-espi-debugger"
 				(path "/df391740-647e-4ab6-9dcd-d61184d66fe9/1d07191d-71e0-43c8-9a4f-6404f7e36093"
-					(reference "R?")
+					(reference "R4019")
 					(unit 1)
 				)
@@
 		(in_pos_files yes)
 		(dnp no)
-		(property "Reference" "R?"
+		(property "Reference" "R4008"
 			(at 107.442 92.71 0)
 			(show_name no)
@@
 			(project "machxo5-espi-debugger"
 				(path "/df391740-647e-4ab6-9dcd-d61184d66fe9/1d07191d-71e0-43c8-9a4f-6404f7e36093"
-					(reference "R?")
+					(reference "R4008")
 					(unit 1)
 				)

Commit message: [#103953] sch/pcb: re-annotate components
Parts:
- renumbered C4005 to C46, C4001 to C47, C4007 to C48, C4006 to C49, C4002 to C50, C4008 to C51, C4003 to C52, C4009 to C53, C4004 to C54, C4010 to C55, D4001 to D1, D4003 to D2, D4004 to D3, D4002 to D4, L4001 to L1, L4002 to L2, Q4001 to Q1, Q4002 to Q2, R4016 to R17, R4017 to R18, R4018 to R19, R4012 to R20, R4013 to R21, R4014 to R22, R4015 to R23, R4003 to R24, R4001 to R25, R4004 to R26, R4008 to R27, R4005 to R28, R4010 to R29, R4007 to R30, R4009 to R31, R4019 to R32, R4020 to R33, R4021 to R34, R4022 to R35, R4011 to R36, R4023 to R37, R4002 to R38, R4006 to R39, R4024 to R40, TP4002 to TP4, TP4001 to TP5, TP4003 to TP6, U4002 to U2, U4001 to U3, U4003 to U4
