File: usb_debug.kicad_sch (KiCad schematic)
At the start: 38 parts, among them J7003 Tag-Connect_TC2050-IDC-NL_2x5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, J7004 USB-C_GCT_USB4105-GF-A, U7002 FT2232HL-REEL, Y7001 Resonator_12MHz_KX-7

Commit message: [#103910] Update power section
Parts:
- removed C7014, C7015: C_30p_0402, antmicro-footprints:C_0402_1005Metric, symbol antmicroCapacitors0402:C_30p_0402
- removed R7008, R7014: R_0R_0402, antmicro-footprints:R_0402_1005Metric, symbol antmicroResistors0402:R_0R_0402
- removed R7010, R7011: R_10R_0402, antmicro-footprints:R_0402_1005Metric, symbol Antmicro Symbols:R_10R_0402
- added C7002, C7003: C_18p_0402, antmicro-footprints:C_0402_1005Metric, symbol antmicroCapacitors0402:C_18p_0402
- added R? (x5): R_0R_0402, antmicro-footprints:R_0402_1005Metric, symbol antmicroResistors0402:R_0R_0402
Connections:
- net EC_UART1.RX is gone; now on net EC_UART0.RX: R7016.2
- net EC_UART1.TX is gone; now on net EC_UART0.TX: R7015.2
- net USB_R_D+ is gone; now on net USB_D+: D7001.1, J7004.A6 (D_{A}+), J7004.B6 (D_{B}+)
- net USB_R_D- is gone; now on net USB_D-: D7001.2, J7004.A7 (D_{A}-), J7004.B7 (D_{B}-)
- net +3V3: now also C7021.2, U7002.50 (VREGIN); no longer C7016.2, C7017.2, C7018.2, U7002.12 (VCORE), U7002.37 (VCORE), U7002.64 (VCORE)
- net EC_JTAG.TCK: now also R?.2
- net EC_JTAG.TDI: now also R?.2
- net EC_JTAG.TDO: now also R?.2
- net EC_JTAG.TMS: now also R?.2
- net EC_JTAG.TRST: now also R?.2
- net GND: now also R7009.2, R7012.1, C7002.1, C7003.1; no longer R7009.1, R7013.1
- net ~{RESET}: now also R7012.2, R7013.1; no longer R7012.1, R7013.2
- net at U7002.16 (ADBUS0): now also R?.1
- net VBUS: now reaches J7004.A4 (VBUS), J7004.A9 (VBUS), J7004.B4 (VBUS), J7004.B9 (VBUS)
- net VBUS: now also R7013.2; no longer R7012.2
- net at U7002.6 (REF): now also R7009.1; no longer R7009.2
- net at U7002.2 (OSCI), Y7001.1: now also C7003.2
- net at U7002.17 (ADBUS1): now also R?.1
- net at U7002.18 (ADBUS2): now also R?.1
- net at U7002.19 (ADBUS3): now also R?.1
- net at U7002.21 (ADBUS4): now also R?.1
- net at U7002.3 (OSCO), Y7001.3: now also C7002.2
- net VCC renamed FTDI_1V8
- net FTDI_1V8: now also C7016.2, C7017.2, C7018.2, U7002.12 (VCORE), U7002.37 (VCORE), U7002.64 (VCORE); no longer C7021.2, U7002.50 (VREGIN)
- no-connect marks 33 -> 30
Other:
- title: MachXO5 eSPI Debugger -> eSPI Adapter
- moved on the sheet: R7009

Commit message: [#103910] Complete schematics
Connections:
- net EC_JTAG.TCK renamed JTAG.TCK
- net EC_JTAG.TDI renamed JTAG.TDI
- net EC_JTAG.TDO renamed JTAG.TDO
- net EC_JTAG.TMS renamed JTAG.TMS
- net EC_JTAG.TRST renamed JTAG.TRST
- net EC_UART0.RX renamed UART0.RX
- net EC_UART0.TX renamed UART0.TX
Other:
- title: eSPI Adapter -> MachXO5 eSPI Debugger
Changed lines of the file:
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@@
 	(paper "A4")
 	(title_block
-		(title "eSPI Adapter")
-		(date "2026-08-21")
+		(title "MachXO5 eSPI Debugger")
+		(date "2026-08-26")
 		(rev "1.0.0")
 		(company "Antmicro")
@@
 		)
 	)
-	(label "EC_JTAG.TDO"
+	(label "JTAG.TDO"
 		(at 255.27 87.63 180)
 		(effects
@@
 		)
 	)
-	(label "EC_JTAG.TMS"
+	(label "JTAG.TMS"
 		(at 255.27 90.17 180)
 		(effects
@@
 		)
 	)
-	(label "EC_JTAG.TMS"
+	(label "JTAG.TMS"
 		(at 35.56 41.91 0)
 		(effects
@@
 		)
 	)
-	(label "EC_UART0.RX"
+	(label "UART0.RX"
 		(at 248.92 153.67 0)
 		(effects
@@
 		)
 	)
-	(label "EC_JTAG.TRST"
+	(label "JTAG.TRST"
 		(at 99.06 39.37 0)
 		(effects
@@
 		)
 	)
-	(label "EC_JTAG.TMS"
+	(label "JTAG.TMS"
 		(at 181.61 49.53 180)
 		(effects
@@
 		)
 	)
-	(label "EC_JTAG.TDI"
+	(label "JTAG.TDI"
 		(at 181.61 41.91 180)
 		(effects
@@
 		)
 	)
-	(label "EC_JTAG.TCK"
+	(label "JTAG.TCK"
 		(at 181.61 46.99 180)
 		(effects
@@
 		)
 	)
-	(label "EC_JTAG.TCK"
+	(label "JTAG.TCK"
 		(at 35.56 46.99 0)
 		(effects
@@
 		)
 	)
-	(label "EC_JTAG.TDI"
+	(label "JTAG.TDI"
 		(at 255.27 85.09 180)
 		(effects
@@
 		)
 	)
-	(label "EC_UART0.TX"
+	(label "UART0.TX"
 		(at 248.92 151.13 0)
 		(effects
@@
 		)
 	)
-	(label "EC_JTAG.TDI"
+	(label "JTAG.TDI"
 		(at 99.06 44.45 0)
 		(effects
@@
 		)
 	)
-	(label "EC_JTAG.TDO"
+	(label "JTAG.TDO"
 		(at 181.61 44.45 180)
 		(effects
@@
 		)
 	)
-	(label "EC_JTAG.TRST"
+	(label "JTAG.TRST"
 		(at 255.27 92.71 180)
 		(effects
@@
 		)
 	)
-	(label "EC_JTAG.TDO"
+	(label "JTAG.TDO"
 		(at 99.06 49.53 0)
 		(effects
@@
 		)
 	)
-	(label "EC_JTAG.TRST"
+	(label "JTAG.TRST"
 		(at 181.61 39.37 180)
 		(effects
@@
 		)
 	)
-	(label "EC_JTAG.TCK"
+	(label "JTAG.TCK"
 		(at 255.27 82.55 180)
 		(effects
@@
 		)
 	)
-	(hierarchical_label "EC_JTAG{JTAG}"
+	(hierarchical_label "JTAG{JTAG}"
 		(shape bidirectional)
 		(at 262.89 77.47 0)
@@
 		)
 	)
-	(hierarchical_label "EC_UART0{UART}"
+	(hierarchical_label "UART0{UART}"
 		(shape bidirectional)
 		(at 266.7 144.78 0)

Commit message: [#103910] Annotate schematics & Clean ERC
Parts:
- added TP7001, TP7002: TP_1mm_SMD, antmicro-footprints:TP_SMD_1mm, symbol antmicroTestPoints:TP_1mm_SMD
- Y7001: symbol Antmicro Symbols:Resonator_12MHz_KX-7 -> antmicroResonators:Resonator_12MHz_KX-7
- gave numbers to parts that had none: 5
Connections:
- net GND: now also TP7002.1
- net VBUS: now also TP7001.1
- net ~{PWREN}: no longer names the net of U7002.60 (~{PWREN})
- net ~{SUSPEND}: no longer names the net of U7002.36 (~{SUSPEND})
- no-connect marks 30 -> 33

Commit message: [#103953] sch/pcb: re-annotate components
Parts:
- renumbered C7009 to C58, C7013 to C59, C7008 to C60, C7018 to C61, C7012 to C62, C7007 to C63, C7020 to C64, C7017 to C65, C7010 to C66, C7006 to C67, C7003 to C68, C7019 to C69, C7016 to C70, C7011 to C71, C7001 to C72, C7002 to C73, C7021 to C74, D7001 to D16, J7003 to J4, J7004 to J5, R7006 to R67, R7007 to R68, R7013 to R69, R7012 to R70, R7001 to R71, R7002 to R72, R7003 to R73, R7004 to R74, R7005 to R75, R7009 to R76, R7008 to R77, R7010 to R78, R7011 to R79, R7014 to R80, R7017 to R81, R7015 to R82, R7016 to R83, TP7001 to TP7, TP7002 to TP8, U7002 to U7, Y7001 to Y2
