File: usb_debug.kicad_sch (KiCad schematic)
At the start: 41 parts, among them J4 Tag-Connect_TC2050-IDC-NL_2x5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, J5 USB-C_GCT_USB4105-GF-A, U7 FT2232HL-REEL, Y2 Resonator_12MHz_KX-7

Commit message: [#103953] Sch: Update DCDC
Parts:
- added C83: C_4u7_10V_X7T_0402, antmicro-footprints:C_0402_1005Metric, symbol antmicroCapacitors0402:C_4u7_10V_X7T_0402
- added D17: TPD2E009_SOT-9X3, antmicro-footprints:SOT-723, symbol antmicroTVSDiodes:TPD2E009_SOT-9X3
Connections:
- net GND: now also C83.1, D17.3; no longer J4.3
- net VBUS: now also C83.2, D17.1, D17.2
- net ~{RESET}: now also J4.3
Other:
- note added: "Note: TC adapter shorts pin 3 to GND this will keep FTDI in reset"
