File: machxo5-espi-debugger.kicad_sch (KiCad schematic)
At the start: 12 parts

Commit message: [#103910] Update power section
Other:
- sheet Connectors renamed USB Debug
- sheet DC-SCM Interposer connector ports: added none; removed DC_SCM_12V_AUX, DC_SCM_P3V0
- sheet MachXO5 ports: added none; removed DC_SCM_P3V0, EC_UART1{UART}
- sheet Power ports: added VIN; removed DC_SCM_12V_AUX
- sheet USB Debug: file connectors.kicad_sch -> usb_debug.kicad_sch
- sheet USB Debug ports: added VBUS; removed EC_UART1{UART}
Changed lines of the file:
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@@
 	(bus
 		(pts
-			(xy 176.53 104.14) (xy 214.63 104.14)
+			(xy 67.31 96.52) (xy 115.57 96.52)
 		)
 		(stroke
@@
 	(wire
 		(pts
-			(xy 19.05 166.37) (xy 21.59 166.37)
+			(xy 115.57 41.91) (xy 76.2 41.91)
 		)
 		(stroke
@@
 	(wire
 		(pts
-			(xy 67.31 93.98) (xy 93.98 93.98)
+			(xy 19.05 166.37) (xy 21.59 166.37)
 		)
 		(stroke
@@
 	(wire
 		(pts
-			(xy 93.98 45.72) (xy 115.57 45.72)
+			(xy 21.59 151.13) (xy 19.05 151.13)
 		)
 		(stroke
@@
 	(wire
 		(pts
-			(xy 21.59 151.13) (xy 19.05 151.13)
+			(xy 67.31 115.57) (xy 91.44 115.57)
 		)
 		(stroke
@@
 		)
 	)
-	(wire
-		(pts
-			(xy 93.98 93.98) (xy 93.98 45.72)
-		)
-		(stroke
-			(width 0)
-			(type default)
-		)
-	)
-	(wire
-		(pts
-			(xy 67.31 97.79) (xy 115.57 97.79)
-		)
-		(stroke
-			(width 0)
-			(type default)
-		)
-	)
-	(wire
-		(pts
-			(xy 67.31 90.17) (xy 90.17 90.17)
-		)
-		(stroke
-			(width 0)
-			(type default)
-		)
-	)
 	(bus
 		(pts
-			(xy 176.53 107.95) (xy 214.63 107.95)
+			(xy 67.31 93.98) (xy 115.57 93.98)
 		)
 		(stroke
@@
 	(wire
 		(pts
-			(xy 90.17 41.91) (xy 115.57 41.91)
+			(xy 91.44 53.34) (xy 115.57 53.34)
 		)
 		(stroke
@@
 	(bus
 		(pts
-			(xy 67.31 101.6) (xy 115.57 101.6)
+			(xy 67.31 127) (xy 115.57 127)
 		)
 		(stroke
@@
 	(wire
 		(pts
-			(xy 19.05 166.37) (xy 19.05 173.99)
+			(xy 76.2 41.91) (xy 76.2 86.36)
 		)
 		(stroke
@@
 		)
 	)
-	(bus
+	(wire
 		(pts
-			(xy 176.53 100.33) (xy 214.63 100.33)
+			(xy 19.05 166.37) (xy 19.05 173.99)
 		)
 		(stroke
@@
 		)
 	)
+	(wire
+		(pts
+			(xy 76.2 86.36) (xy 67.31 86.36)
+		)
+		(stroke
+			(width 0)
+			(type default)
+		)
+	)
 	(bus
 		(pts
@@
 	(wire
 		(pts
-			(xy 90.17 90.17) (xy 90.17 41.91)
+			(xy 91.44 115.57) (xy 91.44 53.34)
 		)
 		(stroke
@@
 			)
 		)
-		(pin "DC_SCM_12V_AUX" input
-			(at 115.57 45.72 180)
-			(effects
-				(font
-					(size 1.27 1.27)
-				)
-				(justify left)
-			)
-		)
 		(pin "DC_SCM_STBY_EN" input
+			(at 115.57 53.34 180)
+			(effects
+				(font
+					(size 1.27 1.27)
+				)
+				(justify left)
+			)
+		)
+		(pin "VIN" input
 			(at 115.57 41.91 180)
 			(effects
@@
 	)
 	(sheet
-		(at 214.63 96.52)
-		(size 27.94 15.24)
+		(at 40.64 78.74)
+		(size 26.67 22.86)
 		(exclude_from_sim no)
 		(in_bom yes)
@@
 			(color 0 0 0 0)
 		)
-		(property "Sheetname" "Connectors"
-			(at 214.63 95.8084 0)
-			(show_name no)
-			(do_not_autoplace no)
-			(effects
-				(font
-					(size 1.27 1.27)
-				)
-				(justify left bottom)
-			)
-		)
-		(property "Sheetfile" "connectors.kicad_sch"
-			(at 214.63 112.3446 0)
+		(property "Sheetname" "USB Debug"
+			(at 40.64 78.0284 0)
+			(show_name no)
+			(do_not_autoplace no)
+			(effects
+				(font
+					(size 1.27 1.27)
+				)
+				(justify left bottom)
+			)
+		)
+		(property "Sheetfile" "usb_debug.kicad_sch"
+			(at 40.64 102.1846 0)
 			(show_name no)
 			(do_not_autoplace no)
@@
 		)
 		(pin "EC_JTAG{JTAG}" bidirectional
-			(at 214.63 107.95 180)
-			(effects
-				(font
-					(size 1.27 1.27)
-				)
-				(justify left)
+			(at 67.31 96.52 0)
+			(effects
+				(font
+					(size 1.27 1.27)
+				)
+				(justify right)
 			)
 		)
 		(pin "EC_UART0{UART}" bidirectional
-			(at 214.63 100.33 180)
-			(effects
-				(font
-					(size 1.27 1.27)
-				)
-				(justify left)
-			)
-		)
-		(pin "EC_UART1{UART}" bidirectional
-			(at 214.63 104.14 180)
-			(effects
-				(font
-					(size 1.27 1.27)
-				)
-				(justify left)
+			(at 67.31 93.98 0)
+			(effects
+				(font
+					(size 1.27 1.27)
+				)
+				(justify right)
+			)
+		)
+		(pin "VBUS" output
+			(at 67.31 86.36 0)
+			(effects
+				(font
+					(size 1.27 1.27)
+				)
+				(justify right)
 			)
 		)
@@
 		)
 		(pin "EC_ESPI{eSPI}" bidirectional
-			(at 115.57 101.6 180)
+			(at 115.57 127 180)
 			(effects
 				(font
@@
 		)
 		(pin "EC_JTAG{JTAG}" bidirectional
-			(at 176.53 107.95 0)
-			(effects
-				(font
-					(size 1.27 1.27)
-				)
-				(justify right)
+			(at 115.57 96.52 180)
+			(effects
+				(font
+					(size 1.27 1.27)
+				)
+				(justify left)
 			)
 		)
@@
 			)
 		)
-		(pin "DC_SCM_P3V0" input
-			(at 115.57 97.79 180)
-			(effects
-				(font
-					(size 1.27 1.27)
-				)
-				(justify left)
-			)
-		)
 		(pin "EC_UART0{UART}" bidirectional
-			(at 176.53 100.33 0)
-			(effects
-				(font
-					(size 1.27 1.27)
-				)
-				(justify right)
-			)
-		)
-		(pin "EC_UART1{UART}" bidirectional
-			(at 176.53 104.14 0)
-			(effects
-				(font
-					(size 1.27 1.27)
-				)
-				(justify right)
+			(at 115.57 93.98 180)
+			(effects
+				(font
+					(size 1.27 1.27)
+				)
+				(justify left)
 			)
 		)
@@
 	)
 	(sheet
-		(at 40.64 74.93)
-		(size 26.67 50.8)
+		(at 40.64 109.22)
+		(size 26.67 22.86)
 		(exclude_from_sim no)
 		(in_bom yes)
@@
 		)
 		(property "Sheetname" "DC-SCM Interposer connector"
-			(at 40.64 74.2184 0)
+			(at 40.64 108.5084 0)
 			(show_name no)
 			(do_not_autoplace no)
@@
 		)
 		(property "Sheetfile" "dc-scm-interposer-connector.kicad_sch"
-			(at 40.64 126.3146 0)
+			(at 40.64 133.1726 0)
 			(show_name no)
 			(do_not_autoplace no)
@@
 			)
 		)
-		(pin "DC_SCM_12V_AUX" output
-			(at 67.31 93.98 0)
+		(pin "EC_ESPI{eSPI}" bidirectional
+			(at 67.31 127 0)
 			(effects
 				(font
@@
 			)
 		)
-		(pin "EC_ESPI{eSPI}" bidirectional
-			(at 67.31 101.6 0)
-			(effects
-				(font
-					(size 1.27 1.27)
-				)
-				(justify right)
-			)
-		)
-		(pin "DC_SCM_P3V0" output
-			(at 67.31 97.79 0)
-			(effects
-				(font
-					(size 1.27 1.27)
-				)
-				(justify right)
-			)
-		)
 		(pin "DC_SCM_STBY_EN" output
-			(at 67.31 90.17 0)
+			(at 67.31 115.57 0)
 			(effects
 				(font
@@
 	)
 	(embedded_fonts no)
-	(embedded_files
-		(file
-			(name "project_table.kicad_wks")
-			(type worksheet)
-			(data |KLUv/WBrDW0WANbgZSAAtxsWHGQdFQ5GzntWK9QpmmWZgOXb7+ug5yaqqhbAiFoAVgBgAFU7yLsP
-				egbhf/yF8Hc4Nk/a13KyB9L8xkUCRuXszoeW5NeKhKtikraf7Pgl/0EDQqL3ccpJK01lQ9eIoaoz
-				fi/7dQ5Bo5Radda+2I7ZR4PubsD4IWlCD7SfQd/3TWr9xRvaWO0Rhypa9Zf8v8emhdWeGIBgKmXw
-				2trvech7Zr8Zgy/27Fl9QCx+7eLbb+98h1eEs9dV/3UQCIN1Tlmb0g6vV027JK29aZvcKu3P3o9V
-				hg7DUUZOya5LVlp16IHWQbNMUi0i6SoUDqNRIBKdAyWo1pQ0uyTW1Npk1fDFkP7ROqNqB72NpWXS
-				6sygSSvFWRAKDXepVDqUoA/+niLnbMr+18E2beyPIg9WmyJMFesZAMJl2CR2GeiUW3ZRidVa55RZ
-				m64XAuGERanEMhHEBCJJoARXrfJqWBATC8c1KtqkHAQR4R7dwi5C+EMRf03Y5EY706rcKn1YOouL
-				by1VaPvdO5VrGuR1BQqpQNhtVpUBfKARrUKKqZkRLWiSYQxQhIiZQZsDSBwY2OZTTnMjBu5vC512
-				vvvDVDtRPoz5X0weovjyAPbS2ZNlE4bfrFc+HCitodaOJlsbZ7cpoIZpGipGACG1pXVwwiPUJCB5
-				B4KPwX/6qzwVDafRsAFCNGb6FBshrlgxqp+9ZCgX1UEIwCC4IeR0pRZt37OiUIRnWIK/j9DOwCC5
-				lSvEr0TMOaaNvm8EZSBhGc+LMU6Zd59V4rCj0m2ag5QIB1Lcx0ikI0PzEQeKC/+VhcalEVA8SCeM
-				JZ4ssnJo/Gxtjw3VMnWyEUNwpXfGDDcv9+Wp5fcoFGMEvrAT25RMSDWHIVaXDtpQ1wPInDpdjYPT
-				fzAeaz4gRt3bJ7J2EbL9tK8WDgOwi95LLocmCk8mlyAiIAT/ELkF0ugQqg==|
-			)
-			(checksum "B3CB3113FBE3DBAF1C1196898B7ACAA6")
-		)
-	)
 )

Commit message: [#103910] Complete schematics
Other:
- removed sheet Flash
- sheet MachXO5 ports: added DONE, FPGA_JTAG{JTAG}, FPGA_UART{UART}, LED[0..3], LED[4..7], ~{INIT}; removed EC_JTAG{JTAG}, EC_QSPI{QSPI}, EC_UART0{UART}
- sheet Port80 LEDs ports: added DONE, LED[0..3], LED[4..7], ~{INIT}; removed none
- sheet USB Debug ports: added JTAG{JTAG}, UART0{UART}; removed EC_JTAG{JTAG}, EC_UART0{UART}
Changed lines of the file:
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@@
 		(color 0 0 0 0)
 	)
+	(wire
+		(pts
+			(xy 176.53 104.14) (xy 217.17 104.14)
+		)
+		(stroke
+			(width 0)
+			(type default)
+		)
+	)
 	(bus
 		(pts
@@
 	(bus
 		(pts
-			(xy 176.53 121.92) (xy 214.63 121.92)
+			(xy 176.53 101.6) (xy 217.17 101.6)
+		)
+		(stroke
+			(width 0)
+			(type default)
+		)
+	)
+	(bus
+		(pts
+			(xy 176.53 93.98) (xy 217.17 93.98)
 		)
 		(stroke
@@
 		)
 	)
+	(bus
+		(pts
+			(xy 176.53 99.06) (xy 217.17 99.06)
+		)
+		(stroke
+			(width 0)
+			(type default)
+		)
+	)
 	(wire
 		(pts
@@
 	(wire
 		(pts
+			(xy 176.53 106.68) (xy 217.17 106.68)
+		)
+		(stroke
+			(width 0)
+			(type default)
+		)
+	)
+	(wire
+		(pts
 			(xy 19.05 158.75) (xy 19.05 166.37)
 		)
@@
 	(bus
 		(pts
-			(xy 176.53 128.27) (xy 214.63 128.27)
+			(xy 176.53 96.52) (xy 217.17 96.52)
 		)
 		(stroke
@@
 		(pts
 			(xy 76.2 86.36) (xy 67.31 86.36)
-		)
-		(stroke
-			(width 0)
-			(type default)
-		)
-	)
-	(bus
-		(pts
-			(xy 176.53 82.55) (xy 214.63 82.55)
 		)
 		(stroke
@@
 			)
 		)
-		(pin "EC_JTAG{JTAG}" bidirectional
+		(pin "JTAG{JTAG}" bidirectional
 			(at 67.31 96.52 0)
 			(effects
@@
 			)
 		)
-		(pin "EC_UART0{UART}" bidirectional
+		(pin "UART0{UART}" bidirectional
 			(at 67.31 93.98 0)
 			(effects
@@
 	)
 	(sheet
-		(at 214.63 118.11)
-		(size 27.94 13.97)
+		(at 217.17 90.17)
+		(size 27.94 21.59)
 		(exclude_from_sim no)
 		(in_bom yes)
@@
 		)
 		(property "Sheetname" "Port80 LEDs"
-			(at 214.63 117.3984 0)
+			(at 217.17 89.4584 0)
 			(show_name no)
 			(do_not_autoplace no)
@@
 		)
 		(property "Sheetfile" "port80-leds.kicad_sch"
-			(at 214.63 132.6646 0)
+			(at 217.17 112.3446 0)
 			(show_name no)
 			(do_not_autoplace no)
@@
 		)
 		(pin "7SEG_H{7SEG}" input
-			(at 214.63 121.92 180)
+			(at 217.17 93.98 180)
 			(effects
 				(font
@@
 		)
 		(pin "7SEG_L{7SEG}" input
-			(at 214.63 128.27 180)
+			(at 217.17 96.52 180)
+			(effects
+				(font
+					(size 1.27 1.27)
+				)
+				(justify left)
+			)
+		)
+		(pin "DONE" input
+			(at 217.17 106.68 180)
+			(effects
+				(font
+					(size 1.27 1.27)
+				)
+				(justify left)
+			)
+		)
+		(pin "LED[0..3]" input
+			(at 217.17 99.06 180)
+			(effects
+				(font
+					(size 1.27 1.27)
+				)
+				(justify left)
+			)
+		)
+		(pin "LED[4..7]" input
+			(at 217.17 101.6 180)
+			(effects
+				(font
+					(size 1.27 1.27)
+				)
+				(justify left)
+			)
+		)
+		(pin "~{INIT}" input
+			(at 217.17 104.14 180)
 			(effects
 				(font
@@
 				(path "/df391740-647e-4ab6-9dcd-d61184d66fe9"
 					(page "6")
-				)
-			)
-		)
-	)
-	(sheet
-		(at 214.63 74.93)
-		(size 27.94 15.24)
-		(exclude_from_sim no)
-		(in_bom yes)
-		(on_board yes)
-		(dnp no)
-		(fields_autoplaced yes)
-		(stroke
-			(width 0.1524)
-			(type solid)
-		)
-		(fill
-			(color 0 0 0 0)
-		)
-		(property "Sheetname" "Flash"
-			(at 214.63 74.2184 0)
-			(show_name no)
-			(do_not_autoplace no)
-			(effects
-				(font
-					(size 1.27 1.27)
-				)
-				(justify left bottom)
-			)
-		)
-		(property "Sheetfile" "flash.kicad_sch"
-			(at 214.63 90.7546 0)
-			(show_name no)
-			(do_not_autoplace no)
-			(effects
-				(font
-					(size 1.27 1.27)
-				)
-				(justify left top)
-			)
-		)
-		(pin "EC_QSPI{QSPI}" bidirectional
-			(at 214.63 82.55 180)
-			(effects
-				(font
-					(size 1.27 1.27)
-				)
-				(justify left)
-			)
-		)
-		(instances
-			(project "machxo5-espi-debugger"
-				(path "/df391740-647e-4ab6-9dcd-d61184d66fe9"
-					(page "5")
 				)
 			)
@@
 			)
 		)
-		(pin "EC_JTAG{JTAG}" bidirectional
+		(pin "7SEG_H{7SEG}" output
+			(at 176.53 93.98 0)
+			(effects
+				(font
+					(size 1.27 1.27)
+				)
+				(justify right)
+			)
+		)
+		(pin "7SEG_L{7SEG}" output
+			(at 176.53 96.52 0)
+			(effects
+				(font
+					(size 1.27 1.27)
+				)
+				(justify right)
+			)
+		)
+		(pin "DONE" output
+			(at 176.53 106.68 0)
+			(effects
+				(font
+					(size 1.27 1.27)
+				)
+				(justify right)
+			)
+		)
+		(pin "FPGA_JTAG{JTAG}" bidirectional
 			(at 115.57 96.52 180)
 			(effects
@@
 			)
 		)
-		(pin "EC_QSPI{QSPI}" bidirectional
-			(at 176.53 82.55 0)
+		(pin "FPGA_UART{UART}" bidirectional
+			(at 115.57 93.98 180)
+			(effects
+				(font
+					(size 1.27 1.27)
+				)
+				(justify left)
+			)
+		)
+		(pin "LED[0..3]" output
+			(at 176.53 99.06 0)
 			(effects
 				(font
@@
 			)
 		)
-		(pin "EC_UART0{UART}" bidirectional
-			(at 115.57 93.98 180)
-			(effects
-				(font
-					(size 1.27 1.27)
-				)
-				(justify left)
-			)
-		)
-		(pin "7SEG_H{7SEG}" output
-			(at 176.53 121.92 0)
+		(pin "LED[4..7]" output
+			(at 176.53 101.6 0)
 			(effects
 				(font
@@
 			)
 		)
-		(pin "7SEG_L{7SEG}" output
-			(at 176.53 128.27 0)
-			(effects
-				(font
+		(pin "~{INIT}" output
+			(at 176.53 104.14 0)
+			(effects
+				(font

Commit message: [#103953] sch/pcb: re-annotate components
Parts:
- renumbered FD1001 to FD1, FD1002 to FD2, FD1003 to FD3, FD1004 to FD4, FD1007 to FD5, FD1008 to FD6, H1001 to H1, H1002 to H2, H1003 to H3, H1004 to H4, N1001 to N1, N1002 to N2
Changed lines of the file:
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@@
 		(dnp no)
 		(fields_autoplaced yes)
-		(property "Reference" "H1002"
+		(property "Reference" "H2"
 			(at 30.48 157.48 0)
 			(show_name no)
@@
 			(project "machxo5-espi-debugger"
 				(path "/df391740-647e-4ab6-9dcd-d61184d66fe9"
-					(reference "H1002")
+					(reference "H2")
 					(unit 1)
 				)
@@
 		(dnp no)
 		(fields_autoplaced yes)
-		(property "Reference" "FD1007"
+		(property "Reference" "FD5"
 			(at 55.88 181.61 0)
 			(show_name no)
@@
 			(project "machxo5-espi-debugger"
 				(path "/df391740-647e-4ab6-9dcd-d61184d66fe9"
-					(reference "FD1007")
+					(reference "FD5")
 					(unit 1)
 				)
@@
 		(dnp no)
 		(fields_autoplaced yes)
-		(property "Reference" "N1001"
+		(property "Reference" "N1"
 			(at 27.94 184.7062 0)
 			(show_name no)
@@
 			(project "machxo5-espi-debugger"
 				(path "/df391740-647e-4ab6-9dcd-d61184d66fe9"
-					(reference "N1001")
+					(reference "N1")
 					(unit 1)
 				)
@@
 		(dnp no)
 		(fields_autoplaced yes)
-		(property "Reference" "H1004"
+		(property "Reference" "H4"
 			(at 30.48 172.72 0)
 			(show_name no)
@@
 			(project "machxo5-espi-debugger"
 				(path "/df391740-647e-4ab6-9dcd-d61184d66fe9"
-					(reference "H1004")
+					(reference "H4")
 					(unit 1)
 				)
@@
 		(dnp no)
 		(fields_autoplaced yes)
-		(property "Reference" "H1003"
+		(property "Reference" "H3"
 			(at 30.48 165.1 0)
 			(show_name no)
@@
 			(project "machxo5-espi-debugger"
 				(path "/df391740-647e-4ab6-9dcd-d61184d66fe9"
-					(reference "H1003")
+					(reference "H3")
 					(unit 1)
 				)
@@
 		(dnp no)
 		(fields_autoplaced yes)
-		(property "Reference" "N1002"
+		(property "Reference" "N2"
 			(at 27.94 192.3262 0)
 			(show_name no)
@@
 			(project "machxo5-espi-debugger"
 				(path "/df391740-647e-4ab6-9dcd-d61184d66fe9"
-					(reference "N1002")
+					(reference "N2")
 					(unit 1)
 				)
@@
 		(dnp no)
 		(fields_autoplaced yes)
-		(property "Reference" "FD1002"
+		(property "Reference" "FD2"
 			(at 55.88 158.75 0)
 			(show_name no)
@@
 			(project "machxo5-espi-debugger"
 				(path "/df391740-647e-4ab6-9dcd-d61184d66fe9"
-					(reference "FD1002")
+					(reference "FD2")
 					(unit 1)
 				)
@@
 		(dnp no)
 		(fields_autoplaced yes)
-		(property "Reference" "#PWR1001"
+		(property "Reference" "#PWR01"
 			(at 27.94 179.07 0)
 			(hide yes)
@@
 			(project "machxo5-espi-debugger"
 				(path "/df391740-647e-4ab6-9dcd-d61184d66fe9"
-					(reference "#PWR1001")
+					(reference "#PWR01")
 					(unit 1)
 				)
@@
 		(dnp no)
 		(fields_autoplaced yes)
-		(property "Reference" "FD1001"
+		(property "Reference" "FD1"
 			(at 55.88 151.13 0)
 			(show_name no)
@@
 			(project "machxo5-espi-debugger"
 				(path "/df391740-647e-4ab6-9dcd-d61184d66fe9"
-					(reference "FD1001")
+					(reference "FD1")
 					(unit 1)
 				)
@@
 		(dnp no)
 		(fields_autoplaced yes)
-		(property "Reference" "FD1008"
+		(property "Reference" "FD6"
 			(at 55.88 189.23 0)
 			(show_name no)
@@
 			(project "machxo5-espi-debugger"
 				(path "/df391740-647e-4ab6-9dcd-d61184d66fe9"
-					(reference "FD1008")
+					(reference "FD6")
 					(unit 1)
 				)
@@
 		(dnp no)
 		(fields_autoplaced yes)
-		(property "Reference" "FD1003"
+		(property "Reference" "FD3"
 			(at 55.88 166.37 0)
 			(show_name no)
@@
 			(project "machxo5-espi-debugger"
 				(path "/df391740-647e-4ab6-9dcd-d61184d66fe9"
-					(reference "FD1003")
+					(reference "FD3")
 					(unit 1)
 				)
@@
 		(dnp no)
 		(fields_autoplaced yes)
-		(property "Reference" "H1001"
+		(property "Reference" "H1"
 			(at 30.48 149.86 0)
 			(show_name no)
@@
 			(project "machxo5-espi-debugger"
 				(path "/df391740-647e-4ab6-9dcd-d61184d66fe9"
-					(reference "H1001")
+					(reference "H1")
 					(unit 1)
 				)
@@
 		(dnp no)
 		(fields_autoplaced yes)
-		(property "Reference" "FD1004"
+		(property "Reference" "FD4"
 			(at 55.88 173.99 0)
 			(show_name no)
@@
 			(project "machxo5-espi-debugger"
 				(path "/df391740-647e-4ab6-9dcd-d61184d66fe9"
-					(reference "FD1004")
+					(reference "FD4")
 					(unit 1)
 				)
