File: machxo5-espi-debugger.kicad_pcb (KiCad board)
At the start: 6 copper layers, 62 x 87 mm, 243 parts, among them J1 PinHeader_2x6_P2.54mm_Drill1.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, J2 PinHeader_2x5_P1.27mm_SMD, J3 PinHeader_2x5_P1.27mm_SMD, J4 Tag-Connect_TC2050-IDC-NL_2x5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, J5 USB-C_GCT_USB4105-GF-A, Q1 DMG1012T-7, Q2 DMG1012T-7, Q3 DMG1012T-7, SW1 SW_KSC441J70SHLFS_SMD, SW2 SW_KSC441J70SHLFS_SMD, U1 LFMXO5-25-7BBG400C, U2 TLV76701_WSON, U3 TPS566231P, U4 TPS566231P, U5 SN74AC7541_VQFN, U6 SN74AC7541_VQFN, U7 FT2232HL-REEL, Y1 Oscillator_125MHz_ASEMB, Y2 Resonator_12MHz_KX-7

Commit message: [#103953] pcb: resolve DRC
Parts:
- moved C4 1.53 mm to (82.5, 107.0), turned to 90 degrees
- moved C18 1.40 mm to (78.2, 104.2), turned to 0 degrees
- moved C13 0.50 mm to (80.3, 101.2)
Routing:
- net +1V8: track 171.0 -> 69.0 mm, vias 18 -> 16
- net /MachXO5/VCC_AUX: track 18.8 -> 3.43 mm
- net /DC-SCM Interposer connector/EC_ESPI.~{RESET}: track 35.3 -> 48.3 mm, vias 3 -> 2
- net /DC-SCM Interposer connector/EC_ESPI.SCK: track 36.6 -> 48.9 mm
- net /MachXO5/VCC_AUXA: track 15.7 -> 3.68 mm
- net /MachXO5/LED5: track 41.2 -> 32.9 mm
- net /MachXO5/VCC_AUXH: track 10.3 -> 2.36 mm
- net /MachXO5/LED4: track 41.4 -> 33.8 mm
- net /MachXO5/~{PROGRAM}: track 28.4 -> 36.0 mm
- net /MachXO5/LED7: track 34.6 -> 27.5 mm, vias 4 -> 2
- net /DC-SCM Interposer connector/EC_ESPI.IO2: track 36.6 -> 42.3 mm
- net /MachXO5/FPGA_JTAG.TRST: track 36.7 -> 41.6 mm, vias 2 -> 0
- net +3V3: track 89.9 -> 86.0 mm
- net GND: track 162.5 -> 158.8 mm, vias 166 -> 159
- net /DC-SCM Interposer connector/EC_ESPI.~{CS0}: track 36.6 -> 33.1 mm
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- added copper zone on In2.Cu, net +1V0
- added copper zone on B.Cu, net +1V8
- added copper zone on In3.Cu, net /MachXO5/VCC_AUX
- added copper zone on B.Cu, net /MachXO5/VCC_AUXA
- added copper zone on In2.Cu, net /MachXO5/VCC_AUXH
- removed copper zone on In2.Cu, net +1V8
- removed copper zone on In4.Cu, net +1V8
