File: machxo5-espi-debugger.kicad_pcb (KiCad board)
At the start: 6 copper layers, 62 x 87 mm, 243 parts, among them J1 PinHeader_2x6_P2.54mm_Drill1.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, J2 PinHeader_2x5_P1.27mm_SMD, J3 PinHeader_2x5_P1.27mm_SMD, J4 Tag-Connect_TC2050-IDC-NL_2x5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, J5 USB-C_GCT_USB4105-GF-A, Q1 DMG1012T-7, Q2 DMG1012T-7, Q3 DMG1012T-7, SW1 SW_KSC441J70SHLFS_SMD, SW2 SW_KSC441J70SHLFS_SMD, U1 LFMXO5-25-7BBG400C, U2 TLV76701_WSON, U3 TPS566231P, U4 TPS566231P, U5 SN74AC7541_VQFN, U6 SN74AC7541_VQFN, U7 FT2232HL-REEL, Y1 Oscillator_125MHz_ASEMB, Y2 Resonator_12MHz_KX-7

Commit message: [#103953] pcb: eSPI length tunning
Routing:
- net /DC-SCM Interposer connector/EC_ESPI.IO2: track 42.3 -> 45.4 mm
- net /DC-SCM Interposer connector/EC_ESPI.IO0: track 33.2 -> 35.5 mm
- net /DC-SCM Interposer connector/EC_ESPI.~{CS0}: track 33.1 -> 35.4 mm
- net /DC-SCM Interposer connector/EC_ESPI.IO3: track 33.3 -> 35.4 mm
- net /DC-SCM Interposer connector/EC_ESPI.IO1: track 34.7 -> 35.6 mm
- net /DC-SCM Interposer connector/EC_ESPI.~{ALERT0}: track 38.8 -> 39.4 mm
